File: fuse-board-large/fuse-board-large.sch (KiCad schematic (older format))
At the start: 26 parts, among them J1 Anderson_two_redblack, J10 Anderson_two_redblack, J11 Anderson_two_redblack, J2 Anderson_two_redblack, J3 Anderson_two_redblack, J4 Anderson_two_redblack, J5 Anderson_two_redblack, J6 Anderson_two_redblack, J7 Anderson_two_redblack, J8 Anderson_two_redblack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

Commit message: fuse-board-large v1.1:
- Update straight Anderson footprint for fixed silk, bigger copper ring
Parts:
- J1: footprint homebrew:Anderson_1337G3_right_angle_bottom_two -> homebrew:Anderson_1336G1_right_angle_bottom_two
Changed lines of the file:
@@
 F 0 "J1" H 1092 1713 60  0000 C CNN
 F 1 "Anderson_two_redblack" H 1092 1819 60  0000 C CNN
-F 2 "homebrew:Anderson_1337G3_right_angle_bottom_two" H 1150 1850 60  0001 C CNN
+F 2 "homebrew:Anderson_1336G1_right_angle_bottom_two" H 1150 1850 60  0001 C CNN
 F 3 "" H 1150 1850 60  0001 C CNN
 	1    1200 2000
