File: distribution-board/anderson_distribution_board.sch (KiCad schematic (older format))
At the start: 5 parts, among them J1 Anderson_two_redblack, J2 Anderson_two_redblack, J3 Anderson_two_redblack, J4 Anderson_two_redblack, J5 Anderson_two_redblack

Commit message: Distribution board v1.1:
- Fix silk on anderson connectors
Parts:
- J2, J3, J4, J5: footprint homebrew:Anderson_1337G3_straight_two -> homebrew:Anderson_1335G1_straight_two
Changed lines of the file:
@@
 EESchema Schematic File Version 4
-LIBS:anderson_distribution_board-cache
-EELAYER 29 0
+EELAYER 30 0
 EELAYER END
 $Descr User 7874 5906
@@
 F 0 "J2" H 2800 1600 60  0000 C CNN
 F 1 "Anderson_two_redblack" H 2800 1900 60  0000 C CNN
-F 2 "homebrew:Anderson_1337G3_straight_two" H 2750 1600 60  0001 C CNN
+F 2 "homebrew:Anderson_1335G1_straight_two" H 2750 1600 60  0001 C CNN
 F 3 "" H 2750 1600 60  0001 C CNN
 	1    2800 1750
@@
 F 0 "J3" H 2800 2050 60  0000 C CNN
 F 1 "Anderson_two_redblack" H 2800 2350 60  0000 C CNN
-F 2 "homebrew:Anderson_1337G3_straight_two" H 2750 2050 60  0001 C CNN
+F 2 "homebrew:Anderson_1335G1_straight_two" H 2750 2050 60  0001 C CNN
 F 3 "" H 2750 2050 60  0001 C CNN
 	1    2800 2200
@@
 F 0 "J5" H 2800 2850 60  0000 C CNN
 F 1 "Anderson_two_redblack" H 2800 3150 60  0000 C CNN
-F 2 "homebrew:Anderson_1337G3_straight_two" H 2750 2850 60  0001 C CNN
+F 2 "homebrew:Anderson_1335G1_straight_two" H 2750 2850 60  0001 C CNN
 F 3 "" H 2750 2850 60  0001 C CNN
 	1    2800 3000
@@
 F 0 "J4" H 2800 2450 60  0000 C CNN
 F 1 "Anderson_two_redblack" H 2800 2750 60  0000 C CNN
-F 2 "homebrew:Anderson_1337G3_straight_two" H 2750 2450 60  0001 C CNN
+F 2 "homebrew:Anderson_1335G1_straight_two" H 2750 2450 60  0001 C CNN
 F 3 "" H 2750 2450 60  0001 C CNN
 	1    2800 2600

Commit message: distribution-board v1.2:
- Update straight Anderson footprint for fixed silk, bigger copper ring
Parts:
- J1: footprint homebrew:Anderson_1337G3_right_angle_bottom_two -> homebrew:Anderson_1336G1_right_angle_bottom_two
Changed lines of the file:
@@
 F 0 "J1" H 1550 1500 60  0000 C CNN
 F 1 "Anderson_two_redblack" H 1550 1800 60  0000 C CNN
-F 2 "homebrew:Anderson_1337G3_right_angle_bottom_two" H 1500 1500 60  0001 C CNN
+F 2 "homebrew:Anderson_1336G1_right_angle_bottom_two" H 1500 1500 60  0001 C CNN
 F 3 "" H 1500 1500 60  0001 C CNN
 	1    1550 1650
